File: MSPM0/TI MSPM0.kicad_pcb (KiCad board)
At the start: 2 copper layers, 37 parts, among them J1 USB_C 4105-GF-A, J2 Conn_ARM_SWD_TagConnect_TC2030, U1 SPX3819M5-L-3-3, U2 CH340E, U3 MSPM0G3507SPTR, U4 LIS2DH, X1 8MHz

Commit message: changes to board stackup and net classes
Parts:
- moved U3 46.6 mm to (100.8, 87.8)
Changed lines of the file:
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@@
 		(0 "F.Cu" signal)
 		(2 "B.Cu" power)
-		(11 "B.Adhes" user "B.Adhesive")
 		(13 "F.Paste" user)
 		(15 "B.Paste" user)
@@
 		(31 "F.CrtYd" user "F.Courtyard")
 		(29 "B.CrtYd" user "B.Courtyard")
-		(33 "B.Fab" user)
 	)
 	(setup
@@
 		(capping no)
 		(filling no)
+		(zone_defaults)
 		(pcbplotparams
 			(layerselection 0x00000000_00000000_55555555_5755f5ff)
@@
 	(footprint "Package_QFP:LQFP-48_7x7mm_P0.5mm"
 		(layer "F.Cu")
-		(at 146.125 98.245)
+		(at 100.75 87.75)
 		(descr "LQFP, 48 Pin (JEDEC MS-026 variation BBC, 1.40mm body thickness, https://www.jedec.org/document_search?search_api_views_fulltext=MS-026, https://www.analog.com/media/en/package-pcb-resources/package/pkg_pdf/ltc-legacy-lqfp/05081760_a_lx48.pdf)")
 		(tags "LQFP QFP CASE-932AA CASE-932-03 C48-1 C48-2 C48-3 C48-5 C48-6 C48-6C PT0048A")

Commit message: starting rough layout
Parts:
- moved J1 91.7 mm to (67.2, 91.0), turned to -90 degrees
- moved U1 85.0 mm to (76.4, 85.0)
- moved D1 82.6 mm to (76.5, 90.5)
- moved MH2 71.4 mm to (67.4, 105.0)
- moved MH1 69.5 mm to (67.0, 78.0)
- moved X1 68.3 mm to (87.5, 97.1)
- moved U2 62.1 mm to (84.0, 90.5)
- moved U4 52.9 mm to (107.8, 97.4)
- moved J2 45.8 mm to (114.8, 90.2)
- moved MH3 27.3 mm to (115.3, 77.6)
- moved MH4 20.6 mm to (116.0, 105.2)
- moved U3 3.62 mm to (98.8, 90.8)
- moved C1 2.60 mm to (143.1, 78.8)
- moved C10 2.60 mm to (147.1, 78.8)
- moved C11 2.60 mm to (163.3, 112.2)
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